File: hardware/chufe-v-0-rev-a/chufe-v-0-rev-a.kicad_pcb (KiCad board)
At the start: 2 copper layers, 50 x 65 mm, 23 parts, among them J1 Conn_02x08_Odd_Even, J2 Conn_01x04_Pin, J3 Barrel_Jack_Switch, Q1 AO3401A, U1 URA2412YMD-20WR3_C5369773, U2 L7805

Commit message: ordenar rev-a
Parts:
- U1: value URA2412YMD-20WR3_C5369773 -> URA2412YMD-20WR3; footprint easyeda2kicad:PWRM-TH_YLPTEC_VRBXXXXYMD-20WR3 -> piruetas:YLPTEC_URA_YMD-20WR3
Changed lines of the file:
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@@
 		)
 	)
-	(footprint "easyeda2kicad:PWRM-TH_YLPTEC_VRBXXXXYMD-20WR3"
+	(footprint "piruetas:YLPTEC_URA_YMD-20WR3"
 		(layer "F.Cu")
 		(at 34.84 55)
@@
 			)
 		)
-		(property "Value" "URA2412YMD-20WR3_C5369773"
+		(property "Value" "URA2412YMD-20WR3"
 			(at 0 14.16 0)
 			(layer "F.Fab")
@@
 			)
 		)
-		(property "Manufacturer" "YLPTEC(易川)"
+		(property "Manufacturer" "YLPTEC"
 			(at 0 0 0)
 			(unlocked yes)
@@
 			)
 		)
-		(attr through_hole)
+(attr through_hole)
 		(duplicate_pad_numbers_are_jumpers no)
-		(fp_line
-			(start -12.7 -12.7)
-			(end -12.7 12.7)
-			(stroke
-				(width 0.25)
-				(type solid)
-			)
-			(layer "F.SilkS")
-		)
-		(fp_line
-			(start -12.7 12.7)
-			(end 12.7 12.7)
-			(stroke
-				(width 0.25)
-				(type solid)
-			)
-			(layer "F.SilkS")
-		)
-		(fp_line
-			(start 12.7 -12.7)
-			(end -12.7 -12.7)
-			(stroke
-				(width 0.25)
-				(type solid)
-			)
-			(layer "F.SilkS")
-		)
-		(fp_line
-			(start 12.7 12.7)
-			(end 12.7 -12.7)
-			(stroke
-				(width 0.25)
-				(type solid)
-			)
-			(layer "F.SilkS")
-		)
-		(fp_circle
-			(center -13.97 -2.67)
-			(end -13.52 -2.67)
-			(stroke
-				(width 0.25)
+		(fp_rect
+			(start -12.82 -12.82)
+			(end 12.82 12.82)
+			(stroke
+				(width 0.12)
 				(type solid)
 			)
@@
 			(layer "F.SilkS")
 		)
-		(fp_circle
-			(center -12.7 -12.7)
-			(end -12.67 -12.7)
-			(stroke
-				(width 0.06)
+		(fp_poly
+			(pts
+				(xy -13.3 -2.54) (xy -14.1 -3.14) (xy -14.1 -1.94)
+			)
+			(stroke
+				(width 0.12)
+				(type solid)
+			)
+			(fill yes)
+			(layer "F.SilkS")
+		)
+		(fp_rect
+			(start -12.95 -12.95)
+			(end 12.95 12.95)
+			(stroke
+				(width 0.05)
 				(type solid)
 			)
 			(fill no)
-			(layer "F.SilkS")
-		)
-		(fp_circle
-			(center -13.97 -2.67)
-			(end -13.67 -2.67)
-			(stroke
-				(width 0.6)
+			(layer "F.CrtYd")
+		)
+		(fp_poly
+			(pts
+				(xy -11.7 -12.7) (xy 12.7 -12.7) (xy 12.7 12.7) (xy -12.7 12.7) (xy -12.7 -11.7)
+			)
+			(stroke
+				(width 0.1)
 				(type solid)
 			)
 			(fill no)
-			(layer "Cmts.User")
-		)
-		(fp_line
-			(start -12.7 -12.7)
-			(end 12.7 -12.7)
-			(stroke
-				(width 0.05)
-				(type solid)
-			)
-			(layer "F.CrtYd")
-		)
-		(fp_line
-			(start -12.7 12.7)
-			(end -12.7 -12.7)
-			(stroke
-				(width 0.05)
-				(type solid)
-			)
-			(layer "F.CrtYd")
-		)
-		(fp_line
-			(start 12.7 -12.7)
-			(end 12.7 12.7)
-			(stroke
-				(width 0.05)
-				(type solid)
-			)
-			(layer "F.CrtYd")
-		)
-		(fp_line
-			(start 12.7 12.7)
-			(end -12.7 12.7)
-			(stroke
-				(width 0.05)
-				(type solid)
-			)
-			(layer "F.CrtYd")
-		)
-		(fp_circle
-			(center -10.16 -10.16)
-			(end -9.91 -10.16)
-			(stroke
-				(width 0.5)
-				(type solid)
-			)
-			(fill no)
-			(layer "F.Fab")
-		)
-		(fp_circle
-			(center -10.16 -2.54)
-			(end -9.91 -2.54)
-			(stroke
-				(width 0.5)
-				(type solid)
-			)
-			(fill no)
-			(layer "F.Fab")
-		)
-		(fp_circle
-			(center -10.16 2.54)
-			(end -9.91 2.54)
-			(stroke
-				(width 0.5)
-				(type solid)
-			)
-			(fill no)
-			(layer "F.Fab")
-		)
-		(fp_circle
-			(center 10.16 -10.16)
-			(end 10.41 -10.16)
-			(stroke
-				(width 0.5)
-				(type solid)
-			)
-			(fill no)
-			(layer "F.Fab")
-		)
-		(fp_circle
-			(center 10.16 0)
-			(end 10.41 0)
-			(stroke
-				(width 0.5)
-				(type solid)
-			)
-			(fill no)
-			(layer "F.Fab")
-		)
-		(fp_circle
-			(center 10.16 10.16)
-			(end 10.41 10.16)
-			(stroke
-				(width 0.5)
-				(type solid)
-			)
-			(fill no)
 			(layer "F.Fab")
 		)
@@
 			)
 		)
-		(pad "1" thru_hole circle
-			(at -10.16 -2.54 90)
-			(size 2.4 2.4)
-			(drill 1.599996)
+		(pad "1" thru_hole rect
+			(at -10.16 -2.54)
+			(size 2.4 2.4)
+			(drill 1.6)
 			(layers "*.Cu" "*.Mask")
 			(remove_unused_layers no)
 			(net "GND")
-			(pinfunction "-VIN_1")
-			(pintype "unspecified")
+			(pinfunction "-VIN")
+			(pintype "power_in")
 		)
 		(pad "2" thru_hole circle
-			(at -10.16 2.54 90)
-			(size 2.4 2.4)
-			(drill 1.599996)
+			(at -10.16 2.54)
+			(size 2.4 2.4)
+			(drill 1.6)
 			(layers "*.Cu" "*.Mask")
 			(remove_unused_layers no)
 			(net "Net-(D1-K)")
-			(pinfunction "+VIN_2")
-			(pintype "unspecified")
+			(pinfunction "+VIN")
+			(pintype "power_in")
 		)
 		(pad "3" thru_hole circle
-			(at 10.16 10.16 90)
-			(size 2.4 2.4)
-			(drill 1.599996)
+			(at 10.16 10.16)
+			(size 2.4 2.4)
+			(drill 1.6)
 			(layers "*.Cu" "*.Mask")
 			(remove_unused_layers no)
 			(net "+12V")
-			(pinfunction "+VO1_3")
-			(pintype "unspecified")
+			(pinfunction "+VO")
+			(pintype "power_out")
 		)
 		(pad "4" thru_hole circle
-			(at 10.16 0 90)
-			(size 2.4 2.4)
-			(drill 1.599996)
+			(at 10.16 0)
+			(size 2.4 2.4)
+			(drill 1.6)
 			(layers "*.Cu" "*.Mask")
 			(remove_unused_layers no)
 			(net "GND")
-			(pinfunction "COM_4")
-			(pintype "unspecified")
+			(pinfunction "COM")
+			(pintype "power_out")
 		)
 		(pad "5" thru_hole circle
-			(at 10.16 -10.16 90)
-			(size 2.4 2.4)
-			(drill 1.599996)
+			(at 10.16 -10.16)
+			(size 2.4 2.4)
+			(drill 1.6)
 			(layers "*.Cu" "*.Mask")
 			(remove_unused_layers no)
 			(net "-12V")
-			(pinfunction "-VO2_5")
-			(pintype "unspecified")
+			(pinfunction "-VO")
+			(pintype "power_out")
 		)
 		(pad "6" thru_hole circle
-			(at -10.16 -10.16 90)
-			(size 2.4 2.4)
-			(drill 1.599996)
+			(at -10.16 -10.16)
+			(size 2.4 2.4)
+			(drill 1.6)
 			(layers "*.Cu" "*.Mask")
 			(remove_unused_layers no)
 			(net "unconnected-(U1-CTRL-Pad6)")
-			(pinfunction "CTRL_6")
-			(pintype "unspecified+no_connect")
+			(pinfunction "CTRL")
+			(pintype "input+no_connect")
 		)
 		(embedded_fonts no)
-		(model "${KIPRJMOD}/../../terceros/easyeda2kicad.3dshapes/PWRM-TH_YLPTEC_VRBXXXXYMD-20WR3.wrl"
+		(model "${KIPRJMOD}/../bibliotecas/piruetas.3dshapes/YLPTEC_URA_YMD-20WR3.wrl"
 			(offset
 				(xyz 0 0 0)
