File: hardware/chufe-v-0-rev-a/chufe-v-0-rev-a.kicad_sch (KiCad schematic)
At the start: 23 parts, among them J1 Conn_02x08_Odd_Even, J2 Conn_01x04_Pin, J3 Barrel_Jack_Switch, Q1 AO3401A, U1 URA2412YMD-20WR3_C5369773, U2 L7805

Commit message: ordenar rev-a
Parts:
- U1: value URA2412YMD-20WR3_C5369773 -> URA2412YMD-20WR3; footprint easyeda2kicad:PWRM-TH_YLPTEC_VRBXXXXYMD-20WR3 -> piruetas:YLPTEC_URA_YMD-20WR3; symbol easyeda2kicad:URA2412YMD-20WR3_C5369773 -> piruetas:URA2412YMD-20WR3; Manufacturer YLPTEC(易川) -> YLPTEC
Changed lines of the file:
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@@
 	)
 	(junction
+		(at 186.69 44.45)
+		(diameter 0)
+		(color 0 0 0 0)
+	)
+	(junction
 		(at 144.78 49.53)
 		(diameter 0)
@@
 	)
 	(symbol
+		(lib_id "power:PWR_FLAG")
+		(at 186.69 44.45 0)
+		(unit 1)
+		(body_style 1)
+		(exclude_from_sim no)
+		(in_bom yes)
+		(on_board yes)
+		(in_pos_files yes)
+		(dnp no)
+		(fields_autoplaced yes)
+		(property "Reference" "#FLG01"
+			(at 186.69 42.55 0)
+			(hide yes)
+			(show_name no)
+			(do_not_autoplace no)
+			(effects
+				(font
+					(size 1.27 1.27)
+				)
+			)
+		)
+		(property "Value" "PWR_FLAG"
+			(at 186.69 40.64 0)
+			(show_name no)
+			(do_not_autoplace no)
+			(effects
+				(font
+					(size 1.27 1.27)
+				)
+			)
+		)
+		(property "Footprint" ""
+			(at 186.69 44.45 0)
+			(hide yes)
+			(show_name no)
+			(do_not_autoplace no)
+			(effects
+				(font
+					(size 1.27 1.27)
+				)
+			)
+		)
+		(property "Datasheet" "~"
+			(at 186.69 44.45 0)
+			(hide yes)
+			(show_name no)
+			(do_not_autoplace no)
+			(effects
+				(font
+					(size 1.27 1.27)
+				)
+			)
+		)
+		(property "Description" "Special symbol for telling ERC where power comes from"
+			(at 186.69 44.45 0)
+			(hide yes)
+			(show_name no)
+			(do_not_autoplace no)
+			(effects
+				(font
+					(size 1.27 1.27)
+				)
+			)
+		)
+		(pin "1"
+		)
+		(instances
+			(project "chufe-v-0-rev-a"
+				(path "/76d7d92c-1316-4bcb-a187-c7124ef49ded"
+					(reference "#FLG01")
+					(unit 1)
+				)
+			)
+		)
+	)
+	(symbol
 		(lib_id "power:GND")
 		(at 252.73 67.31 0)
@@
 	)
 	(symbol
-		(lib_id "easyeda2kicad:URA2412YMD-20WR3_C5369773")
+		(lib_id "piruetas:URA2412YMD-20WR3")
 		(at 205.74 46.99 0)
 		(unit 1)
@@
 			)
 		)
-		(property "Value" "URA2412YMD-20WR3_C5369773"
+		(property "Value" "URA2412YMD-20WR3"
 			(at 205.74 39.37 0)
 			(show_name no)
@@
 			)
 		)
-		(property "Footprint" "easyeda2kicad:PWRM-TH_YLPTEC_VRBXXXXYMD-20WR3"
+		(property "Footprint" "piruetas:YLPTEC_URA_YMD-20WR3"
 			(at 205.74 57.15 0)
 			(hide yes)
@@
 			)
 		)
-		(property "Manufacturer" "YLPTEC(易川)"
+		(property "Manufacturer" "YLPTEC"
 			(at 205.74 62.23 0)
 			(hide yes)
